File: Phaser.kicad_pcb (KiCad board)
At the start: 2 copper layers, 99.4 x 85.1 mm, 51 parts, among them J1 Barrel_Jack, J2 Barrel_Jack, Q1 Q_NJFET_GDS, Q2 Q_NJFET_GDS, Q3 Q_NJFET_GDS, Q4 Q_NJFET_GDS, Q5 2N3904, SW1 SW_DPDT_x2, U1 TL062, U2 TL062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

Commit message: Phaser Edit 1
Parts:
- moved R4 4.44 mm to (124.6, 54.9)
Routing:
- net Net-(C3-Pad1): track 36.1 -> 40.1 mm
- net Net-(R3-Pad2): track 23.1 -> 27.2 mm
Changed lines of the file:
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@@
   )
   (footprint "10kres:RESC6332X70N" (layer "F.Cu")
-    (at 128.27 57.43)
+    (at 124.6124 54.9148)
     (property "Sheetfile" "Phaser.kicad_sch")
     (property "Sheetname" "")
@@
   (segment (start 132.075 66.035) (end 134.9 68.86) (width 0.508) (layer "F.Cu") (net 5))
   (segment (start 134.415 78.31) (end 135.89 78.31) (width 0.508) (layer "F.Cu") (net 5))
-  (segment (start 131.214 57.43) (end 131.214 60.374) (width 0.254) (layer "F.Cu") (net 6))
   (segment (start 145.61392 70.28608) (end 141.12608 70.28608) (width 0.508) (layer "F.Cu") (net 6))
   (segment (start 152.715 69.215) (end 153.439 69.215) (width 0.508) (layer "F.Cu") (net 6))
-  (segment (start 131.214 60.374) (end 137.16 66.32) (width 0.254) (layer "F.Cu") (net 6))
   (segment (start 152.715 69.215) (end 151.53648 68.03648) (width 0.508) (layer "F.Cu") (net 6))
   (segment (start 141.12608 70.28608) (end 137.16 66.32) (width 0.508) (layer "F.Cu") (net 6))
+  (segment (start 131.214 60.374) (end 137.16 66.32) (width 0.254) (layer "F.Cu") (net 6))
   (segment (start 153.439 69.215) (end 157.249 73.025) (width 0.508) (layer "F.Cu") (net 6))
   (segment (start 151.53648 68.03648) (end 147.86352 68.03648) (width 0.508) (layer "F.Cu") (net 6))
+  (segment (start 127.5564 54.9148) (end 131.214 58.5724) (width 0.254) (layer "F.Cu") (net 6))
   (segment (start 147.86352 68.03648) (end 145.61392 70.28608) (width 0.508) (layer "F.Cu") (net 6))
+  (segment (start 131.214 58.5724) (end 131.214 60.374) (width 0.254) (layer "F.Cu") (net 6))
   (segment (start 149.0625 80.0975) (end 151.13 78.03) (width 0.508) (layer "F.Cu") (net 7))
   (segment (start 150.815 69.215) (end 150.815 69.53) (width 0.508) (layer "F.Cu") (net 7))
@@
   (segment (start 111.529 130.579) (end 111.529 128.27) (width 0.254) (layer "F.Cu") (net 18))
   (segment (start 134.62 128.27) (end 139.1025 123.7875) (width 0.508) (layer "F.Cu") (net 18))
+  (segment (start 125.326 58.5724) (end 125.326 61.364) (width 0.508) (layer "F.Cu") (net 19))
+  (segment (start 124.46 62.23) (end 124.46 64.765) (width 0.508) (layer "F.Cu") (net 19))
   (segment (start 137.16 71.4) (end 135.535 71.4) (width 0.508) (layer "F.Cu") (net 19))
   (segment (start 127.005 67.31) (end 124.46 64.765) (width 0.508) (layer "F.Cu") (net 19))
+  (segment (start 121.6684 54.9148) (end 125.326 58.5724) (width 0.508) (layer "F.Cu") (net 19))
   (segment (start 125.326 61.364) (end 124.46 62.23) (width 0.508) (layer "F.Cu") (net 19))
-  (segment (start 124.46 62.23) (end 124.46 64.765) (width 0.508) (layer "F.Cu") (net 19))
-  (segment (start 125.326 57.43) (end 125.326 61.364) (width 0.508) (layer "F.Cu") (net 19))
   (segment (start 131.445 67.31) (end 127.005 67.31) (width 0.508) (layer "F.Cu") (net 19))
   (segment (start 135.535 71.4) (end 131.445 67.31) (width 0.508) (layer "F.Cu") (net 19))
@@
   (segment (start 99.06 127) (end 102.235 127) (width 0.508) (layer "F.Cu") (net 31))
   (segment (start 102.235 127) (end 106.045 123.19) (width 0.508) (layer "F.Cu") (net 31))
-  (zone (net 1) (net_name "GND") (layer "F.Cu") (hatch edge 0.508)
-    (connect_pads (clearance 0.508))
-    (min_thickness 0.254) (filled_areas_thickness no)
-    (fill yes (thermal_gap 0.508) (thermal_bridge_width 0.508))
-    (polygon
-      (pts
-        (xy 96.6216 50.1904)
-        (xy 190.8048 50.1904)
-        (xy 190.8048 129.286)
-        (xy 184.8104 135.2804)
-        (xy 97.4852 135.2804)
-        (xy 94.1832 131.9784)
-        (xy 91.44 129.2352)
-        (xy 91.44 50.1396)
-        (xy 96.6216 50.1396)
-      )
-    )
-  )
   (zone (net 1) (net_name "GND") (layers F&B.Cu) (name "Ground Plane") (hatch edge 0.508)
     (connect_pads (clearance 0.508))
     (min_thickness 0.254) (filled_areas_thickness no)
-    (fill yes (thermal_gap 0.508) (thermal_bridge_width 0.508))
+    (fill yes (thermal_gap 0.508) (thermal_bridge_width 0.508) (island_removal_mode 1) (island_area_min 0))
     (polygon
       (pts
